Commit message: trying to visualize lidar in rviz

File: resource/custom_robot.urdf (robot description, URDF)
Before this commit: robot custom_robot, 1 links, 0 joints
Links:
- added link lds0_link
Joints:
- added joint lds0_joint: type fixed, parent base_link, child lds0_link, origin xyz=0 0 0 rpy=0 0 0

Commit message: Fixed remapping issue for cmd_vel and test_vel

File: resource/custom_robot.urdf (robot description, URDF)
Before this commit: robot custom_robot, 0 links, 0 joints
Links:
- added link base_link
- added link lidar_frame
Joints:
- added joint lidar_joint: type fixed, parent base_link, child lidar_frame, origin xyz=0 0 0.1 rpy=0 0 0
